File: KiCAD/arduTester/arduTester.kicad_pcb (KiCad board)
At the start: 2 copper layers, 113.7 x 61 mm, 14 parts, among them J1 3-pin_test_header, J2 2-pin_power_input_header, J3 3-pin_test_header, SW1 SW_Push, U1 LCD_HD44780

Commit message: forgot resistor
Connections:
- A1 pad 5: Net-(A1-Pad5) -> +5V

Commit message: mini pro
Parts:
- added R8: 10k, My_Misc:R_Axial_DIN0207_L6.3mm_D2.5mm_P10.16mm_Horizontal_larger_pads, F.Cu at (225.4, 89.5)
- moved SW1 13.5 mm to (248.7, 71.0), turned to 180 degrees
Connections:
- A1 pad 12: +5V -> Net-(A1-Pad12)
- SW1 pad 1: +5V -> Net-(A1-Pad12)
Routing:
- net +5V: track 274.8 -> 109.0 mm
- net Net-(A1-Pad12): track 0.00 -> 64.6 mm
- net Net-(A1-Pad8): track 50.5 -> 55.7 mm
- net GND: track 221.5 -> 223.0 mm

Commit message: Schematics and PCB. Scad
Parts:
- added C1: 1n, My_Misc:CP_Radial_D5.0mm_P2.00mm_larger, F.Cu at (166.4, 64.8)
- added SW2: SW_Push, My_Misc:SW_PUSH_6mm_large, F.Cu at (170.8, 108.0)
Connections:
- A1 pad 6: Net-(A1-Pad6) -> GND
- A1 pad 7: Net-(A1-Pad7) -> GND
Routing:
- net GND: track 223.0 -> 297.5 mm
- net Net-(A1-Pad3): track 0.00 -> 25.6 mm
- net Net-(A1-Pad30): track 0.00 -> 13.6 mm
- net TP1: track 88.0 -> 86.5 mm
- net Net-(A1-Pad26): track 36.3 -> 35.2 mm
- net Net-(A1-Pad25): track 41.5 -> 40.5 mm
- net Net-(A1-Pad12): track 64.6 -> 64.0 mm

Commit message: schematics
Parts:
- C1: footprint My_Misc:CP_Radial_D5.0mm_P2.00mm_larger -> My_Misc:C_Disc_D3.0mm_W1.6mm_P2.50mm_larg
- moved C1 1.80 mm to (167.6, 63.5), turned to 180 degrees
Routing:
- net GND: track 297.5 -> 298.5 mm

Commit message: kicad6
Parts:
- A1: footprint My_Arduino:Arduino_UNO_R3_shield_larger_pads -> My_Arduino:Arduino_UNO_R3_shield_large
- U1: footprint My_Parts:LCD_16x2_large -> My_Parts:LCD_HD44780_16x2_w_headers_large
- moved A1 49.1 mm to (173.1, 63.5)
Connections:
- A1 pad 1: Net-(A1-Pad1) -> unconnected-(A1-Pad1)
- A1 pad 13: Net-(A1-Pad13) -> unconnected-(A1-Pad13)
- A1 pad 14: Net-(A1-Pad14) -> unconnected-(A1-Pad14)
- A1 pad 15: Net-(A1-Pad15) -> unconnected-(A1-Pad15)
- A1 pad 16: Net-(A1-Pad16) -> unconnected-(A1-Pad16)
- A1 pad 2: Net-(A1-Pad2) -> unconnected-(A1-Pad2)
- A1 pad 31: Net-(A1-Pad31) -> unconnected-(A1-Pad31)
- A1 pad 32: Net-(A1-Pad32) -> unconnected-(A1-Pad32)
- A1 pad 4: Net-(A1-Pad4) -> unconnected-(A1-Pad4)
- U1 pad 10: Net-(U1-Pad10) -> unconnected-(U1-Pad10)
- U1 pad 7: Net-(U1-Pad7) -> unconnected-(U1-Pad7)
- U1 pad 8: Net-(U1-Pad8) -> unconnected-(U1-Pad8)
- U1 pad 9: Net-(U1-Pad9) -> unconnected-(U1-Pad9)
Routing:
- net +5V: track 109.0 -> 106.1 mm
- net TP2: track 141.9 -> 139.5 mm
- net GND: track 298.5 -> 300.9 mm
- net TP3: track 112.9 -> 115.0 mm
- net TP1: track 86.5 -> 84.7 mm
- net Net-(A1-Pad8): track 55.4 -> 54.6 mm
- net Net-(A1-Pad25): track 40.5 -> 39.9 mm
- net Net-(A1-Pad23): track 51.1 -> 50.5 mm
- net Net-(A1-Pad24): track 46.0 -> 45.3 mm
- net Net-(A1-Pad28): track 28.2 -> 27.7 mm
Other:
- net class Default removed
