File: KiCAD/arduTesterMiniPro/arduTesterMiniPro.kicad_pcb (KiCad board)
At the start: 2 copper layers, 123.8 x 57.1 mm, 19 parts, among them J1 3-pin_test_header, J2 3-pin_test_header, J3 2-pin_power_input_header, SW1 SW_Push, U1 LCD_HD44780, U2 Arduino_Mini_Pro

Commit message: mini pro
Parts:
- removed the REF** at (108.6, 71.1)
- removed the REF** at (197.5, 62.2)
- removed the REF** at (225.4, 113.0)
- removed the REF** at (108.0, 113.0)
- added REF**: MountingHole_3.2mm_M3, MountingHole:MountingHole_3.2mm_M3, F.Cu at (108.0, 71.1)
- added REF**: MountingHole_3.2mm_M3, MountingHole:MountingHole_3.2mm_M3, F.Cu at (196.8, 62.2)
- added REF**: MountingHole_3.2mm_M3, MountingHole:MountingHole_3.2mm_M3, F.Cu at (226.1, 113.7)
- added REF**: MountingHole_3.2mm_M3, MountingHole:MountingHole_3.2mm_M3, F.Cu at (108.0, 113.7)
Routing:
- net GND: track 307.6 -> 304.5 mm
Other:
- board size 123.8 x 57.1 mm -> 124.5 x 57.8 mm
- net class Default: clearance 0.762 -> 1.016
- rule trace_clearance: 0.762 -> 1.016

Commit message: schematics
Parts:
- removed REF** (x4): MountingHole_3.2mm_M3, MountingHole:MountingHole_3.2mm_M3
- added SW2: SW_Push, My_Misc:SW_PUSH_6mm_large, F.Cu at (184.2, 72.4)
- moved R2 13.6 mm to (185.4, 83.8)
- moved R1 13.6 mm to (155.6, 73.0)
- moved R5 13.6 mm to (212.1, 106.0)
- moved R6 13.6 mm to (201.9, 101.0)
- moved R7 13.6 mm to (212.1, 95.9)
- moved R8 13.6 mm to (201.9, 90.8)
- moved J1 13.6 mm to (196.2, 113.0)
- moved J2 13.6 mm to (200.9, 113.0)
- moved J3 13.6 mm to (193.0, 70.5)
- moved R3 13.6 mm to (188.0, 113.0)
- moved R4 13.6 mm to (177.8, 118.1)
- moved RV1 13.6 mm to (132.7, 110.5)
- moved SW1 13.6 mm to (210.2, 70.5)
- moved U1 13.6 mm to (101.3, 71.2)
- moved U2 13.6 mm to (176.5, 74.8)
Routing:
- net Net-(SW2-Pad1): track 0.00 -> 22.1 mm
- net GND: track 304.5 -> 318.3 mm, vias 2 -> 0
Other:
- board text removed: "GND"

Commit message: kicad6
Parts:
- U1: footprint My_Parts:LCD_16x2_large -> My_Parts:LCD_HD44780_16x2_w_headers_large
- moved U2 4.10 mm to (177.7, 78.7)
Connections:
- U1 pad 10: Net-(U1-Pad10) -> unconnected-(U1-Pad10)
- U1 pad 7: Net-(U1-Pad7) -> unconnected-(U1-Pad7)
- U1 pad 8: Net-(U1-Pad8) -> unconnected-(U1-Pad8)
- U1 pad 9: Net-(U1-Pad9) -> unconnected-(U1-Pad9)
- U2 pad 1: Net-(U2-Pad1) -> unconnected-(U2-Pad1)
- U2 pad 2: Net-(U2-Pad2) -> unconnected-(U2-Pad2)
- U2 pad 3: Net-(U2-Pad3) -> unconnected-(U2-Pad3)
Routing:
- net GND: track 318.3 -> 313.1 mm
- net TP1: track 37.1 -> 41.2 mm
- net +5V: track 166.4 -> 164.6 mm
- net TP3: track 61.8 -> 60.3 mm
- net Net-(SW2-Pad1): track 22.1 -> 21.0 mm
- net TP2: track 68.7 -> 67.6 mm
- net Net-(U1-Pad4): track 90.7 -> 89.7 mm
- net Net-(R2-Pad2): track 42.5 -> 41.5 mm
Other:
- net class Default removed
