File: KiCAD/arduTester-SMD/arduTester-SMD.kicad_sch (KiCad schematic)
At the start: 17 parts, among them J1 3-pin_test_header, J2 2-pin_power_input_header, J3 3-pin_test_header, SW1 SW_Push, SW2 SW_Push, U1 LCD_HD44780

Commit message: kicad version
Other:
- added sheet atmega (atmega.kicad_sch)
Changed lines of the file:
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@@
+		)
+	)
+	(sheet
+		(at 255.27 151.13)
+		(size 12.7 3.81)
+		(fields_autoplaced yes)
+		(stroke
+			(width 0.1524)
+			(type solid)
+		)
+		(fill
+			(color 0 0 0 0.0000)
+		)
+		(property "Sheetname" "atmega"
+			(at 255.27 150.4184 0)
+			(effects
+				(font
+					(size 1.27 1.27)
+				)
+				(justify left bottom)
+			)
+		)
+		(property "Sheetfile" "atmega.kicad_sch"
+			(at 255.27 155.5246 0)
+			(effects
+				(font
+					(size 1.27 1.27)
+				)
+				(justify left top)
+			)
+		)
+		(property "Field2" ""
+			(at 255.27 151.13 0)
+			(effects
+				(font
+					(size 1.27 1.27)
+				)
+				(hide yes)
+			)
+		)
+		(instances
+			(project "arduTester-SMD"
+				(path "/46fbff5f-5f07-426e-abff-92611b77fb42"
+					(page "2")
+				)
+			)
 		)
 	)
